Commit message: add camera roughly

File: urdf/ee/openarm_hand.xacro (robot description, xacro)
@@ -2,5 +2,5 @@
 <robot xmlns:xacro="http://www.ros.org/wiki/xacro" name="hand">
   <!-- safety_distance: Minimum safety distance in [m] by which the collision volumes are expanded and which is enforced during robot motions -->
-  <xacro:macro name="openarm_hand" params="connected_to:='' arm_type arm_prefix:='' ee_type ee_inertials ee_kinematics_link rpy_ee:='0 0 0' xyz_ee:='0 0 0' tcp_xyz:='0 0 0' tcp_rpy:='0 0 0' description_pkg:=openarm_description">
+  <xacro:macro name="openarm_hand" params="connected_to:='' arm_type arm_prefix:='' ee_type ee_inertials ee_kinematics_link rpy_ee:='0 0 0' xyz_ee:='0 0 0' tcp_xyz:='0 0 0' tcp_rpy:='0 0 0' description_pkg:='openarm_description'">
     <xacro:property name="ee_prefix" default=""/>
     <xacro:unless value="${arm_type == ''}">

File: urdf/robot/openarm_robot.xacro (robot description, xacro)
@@ -28,12 +28,18 @@
             body_connected_to='world'
             bimanual:=false
-            right_arm_base_xyz='0 0 0'
-            left_arm_base_xyz='0 0 0'
-            right_arm_base_rpy='0 0 0'
-            left_arm_base_rpy='0 0 0'
+            right_arm_base_xyz:='0 0 0'
+            left_arm_base_xyz:='0 0 0'
+            right_arm_base_rpy:='0 0 0'
+            left_arm_base_rpy:='0 0 0'
             left_can_interface:='can1'
             right_can_interface:='can0'
             left_arm_prefix:='left_'
             right_arm_prefix:='right_'
+            left_wrist_camera:='false'
+            right_wrist_camera:='false'
+            left_wrist_cam_xyz:='0 0 0'
+            left_wrist_cam_rpy:='0 0 0'
+            right_wrist_cam_xyz:='0 0 0'
+            right_wrist_cam_rpy:='0 0 0'
             can_fd:='true'
             "
@@ -49,4 +55,7 @@
     <xacro:if value="${ee_type != 'none'}">
         <xacro:include filename="$(find openarm_description)/urdf/ee/${ee_type}_arguments.xacro" />
+    </xacro:if>
+    <xacro:if value="${left_wrist_camera or right_wrist_camera}">
+        <xacro:include filename="$(find realsense2_description)/urdf/_d405.urdf.xacro"/>
     </xacro:if>
     <xacro:property name="arm_prefix_modified" value="${'' if arm_prefix == '' else arm_prefix + '_'}" />
@@ -78,4 +87,15 @@
         kinematics_link="${kinematics_link}"
         kinematics_offset="${kinematics_offset}" />
+        <xacro:if value="${left_wrist_camera}">
+            <link name="openarm_left_camera_mount"/>
+            <joint name="openarm_left_camera_mount_joint" type="fixed">
+              <parent link="openarm_left_link7"/>
+              <child link="openarm_left_camera_mount"/>
+              <origin xyz="${left_wrist_cam_xyz}" rpy="${left_wrist_cam_rpy}"/>
+            </joint>
+            <xacro:sensor_d405 parent="openarm_left_camera_mount" name="left_realsense" use_nominal_extrinsics="true">
+              <origin xyz="0 0 0" rpy="0 0 0"/>
+            </xacro:sensor_d405>
+        </xacro:if>
         <!-- right arm -->
         <xacro:openarm_arm
@@ -92,4 +112,15 @@
         kinematics_link="${kinematics_link}"
         kinematics_offset="${kinematics_offset}" />
+        <xacro:if value="${right_wrist_camera}">
+            <link name="openarm_right_camera_mount"/>
+            <joint name="openarm_right_camera_mount_joint" type="fixed">
+              <parent link="openarm_right_link7"/>
+              <child link="openarm_right_camera_mount"/>
+              <origin xyz="${right_wrist_cam_xyz}" rpy="${right_wrist_cam_rpy}"/>
+            </joint>
+            <xacro:sensor_d405 parent="openarm_right_camera_mount" name="right_realsense" use_nominal_extrinsics="true">
+              <origin xyz="0.1 0 0" rpy="0 0 0"/>
+            </xacro:sensor_d405>
+        </xacro:if>
         <!-- ros2_control hardware interfaces for bimanual setup -->
         <xacro:if value="${ros2_control}">

File: urdf/robot/v10.urdf.xacro (robot description, xacro)
@@ -26,4 +26,10 @@
   <xacro:arg name="left_arm_base_xyz" default="0.0 0.031 0.698" />
   <xacro:arg name="left_arm_base_rpy" default="-1.5708 0 0" />
+  <xacro:arg name="left_wrist_camera" default="true"/>
+  <xacro:arg name="right_wrist_camera" default="true"/>
+  <xacro:arg name="left_wrist_cam_xyz" default="0 0 0"/>
+  <xacro:arg name="left_wrist_cam_rpy" default="0 0 0"/>
+  <xacro:arg name="right_wrist_cam_xyz" default="0 0 0"/>
+  <xacro:arg name="right_wrist_cam_rpy" default="0 0 0"/>
   <xacro:arg name="can_fd" default="true" />
   <xacro:openarm_robot
@@ -59,4 +65,10 @@
   right_arm_base_rpy="$(arg right_arm_base_rpy)"
   left_arm_base_rpy="$(arg left_arm_base_rpy)"
+  left_wrist_camera="$(arg left_wrist_camera)"
+  right_wrist_camera="$(arg right_wrist_camera)"
+  left_wrist_cam_xyz="$(arg left_wrist_cam_xyz)"
+  right_wrist_cam_xyz="$(arg right_wrist_cam_xyz)"
+  left_wrist_cam_rpy="$(arg left_wrist_cam_rpy)"
+  right_wrist_cam_rpy="$(arg right_wrist_cam_rpy)"
   can_fd="$(arg can_fd)"
   />
