Commit message: add: chest camera

File: urdf/robot/openarm_robot.xacro (robot description, xacro)
@@ -42,4 +42,7 @@
             right_wrist_cam_xyz:='0 0 0'
             right_wrist_cam_rpy:='0 0 0'
+            body_camera='false'
+            body_cam_xyz='0 0 0'
+            body_cam_rpy='0 0 0'
             can_fd:='true'
             "
@@ -58,4 +61,7 @@
     <xacro:if value="${left_wrist_camera or right_wrist_camera}">
         <xacro:include filename="$(find realsense2_description)/urdf/_d405.urdf.xacro"/>
+    </xacro:if>
+    <xacro:if value="${body_camera}">
+        <xacro:include filename="$(find realsense2_description)/urdf/_d435.urdf.xacro"/>
     </xacro:if>
     <xacro:property name="arm_prefix_modified" value="${'' if arm_prefix == '' else arm_prefix + '_'}" />
@@ -87,4 +93,15 @@
         kinematics_link="${kinematics_link}"
         kinematics_offset="${kinematics_offset}" />
+        <xacro:if value="${body_camera}">
+            <link name="openarm_body_camera_mount"/>
+            <joint name="openarm_body_camera_mount_joint" type="fixed">
+              <parent link="openarm_body_link0"/>
+              <child link="openarm_body_camera_mount"/>
+              <origin xyz="0 0 0" rpy="0 0 0"/>
+            </joint>
+            <xacro:sensor_d435 parent="openarm_body_camera_mount" name="body_realsense" use_nominal_extrinsics="true">
+              <origin xyz="${body_cam_xyz}" rpy="${body_cam_rpy}"/>
+            </xacro:sensor_d435>
+        </xacro:if>
         <xacro:if value="${left_wrist_camera}">
             <link name="openarm_left_camera_mount"/>
@@ -92,8 +109,8 @@
               <parent link="openarm_left_link7"/>
               <child link="openarm_left_camera_mount"/>
-              <origin xyz="${left_wrist_cam_xyz}" rpy="${left_wrist_cam_rpy}"/>
+              <origin xyz="0 0 0" rpy="0 0 0"/>
             </joint>
             <xacro:sensor_d405 parent="openarm_left_camera_mount" name="left_realsense" use_nominal_extrinsics="true">
-              <origin xyz="0 0 0" rpy="0 0 0"/>
+              <origin xyz="${left_wrist_cam_xyz}" rpy="${left_wrist_cam_rpy}"/>
             </xacro:sensor_d405>
         </xacro:if>
@@ -117,8 +134,8 @@
               <parent link="openarm_right_link7"/>
               <child link="openarm_right_camera_mount"/>
-              <origin xyz="${right_wrist_cam_xyz}" rpy="${right_wrist_cam_rpy}"/>
+              <origin xyz="0 0 0" rpy="0 0 0"/>
             </joint>
             <xacro:sensor_d405 parent="openarm_right_camera_mount" name="right_realsense" use_nominal_extrinsics="true">
-              <origin xyz="0.1 0 0" rpy="0 0 0"/>
+              <origin xyz="${right_wrist_cam_xyz}" rpy="${right_wrist_cam_rpy}"/>
             </xacro:sensor_d405>
         </xacro:if>

File: urdf/robot/v10.urdf.xacro (robot description, xacro)
@@ -28,8 +28,11 @@
   <xacro:arg name="left_wrist_camera" default="true"/>
   <xacro:arg name="right_wrist_camera" default="true"/>
-  <xacro:arg name="left_wrist_cam_xyz" default="0 0 0"/>
+  <xacro:arg name="left_wrist_cam_xyz" default="0.1 0 0"/>
   <xacro:arg name="left_wrist_cam_rpy" default="0 0 0"/>
-  <xacro:arg name="right_wrist_cam_xyz" default="0 0 0"/>
+  <xacro:arg name="right_wrist_cam_xyz" default="0.1 0 0"/>
   <xacro:arg name="right_wrist_cam_rpy" default="0 0 0"/>
+  <xacro:arg name="body_camera" default="true"/>
+  <xacro:arg name="body_cam_xyz" default="0.05 0 0.63"/>
+  <xacro:arg name="body_cam_rpy" default="0 ${pi / 6.0} 0"/>
   <xacro:arg name="can_fd" default="true" />
   <xacro:openarm_robot
@@ -71,4 +74,7 @@
   left_wrist_cam_rpy="$(arg left_wrist_cam_rpy)"
   right_wrist_cam_rpy="$(arg right_wrist_cam_rpy)"
+  body_camera="$(arg body_camera)"
+  body_cam_xyz="$(arg body_cam_xyz)"
+  body_cam_rpy="$(arg body_cam_rpy)"
   can_fd="$(arg can_fd)"
   />

Commit message: chest camera

File: urdf/robot/openarm_robot.xacro (robot description, xacro)
@@ -45,4 +45,8 @@
             body_cam_xyz='0 0 0'
             body_cam_rpy='0 0 0'
+            chest_camera:='false'
+            chest_cam_xyz:='0.055 0.045 0.68'
+            chest_cam_rpy:='-2.40 0.03 -1.605'
+            chest_camera_parent:='openarm_link0'
             can_fd:='true'
             "
@@ -62,5 +66,5 @@
         <xacro:include filename="$(find realsense2_description)/urdf/_d405.urdf.xacro"/>
     </xacro:if>
-    <xacro:if value="${body_camera}">
+    <xacro:if value="${body_camera or chest_camera}">
         <xacro:include filename="$(find realsense2_description)/urdf/_d435.urdf.xacro"/>
     </xacro:if>
@@ -225,4 +229,15 @@
         </xacro:if>
         </xacro:if>
+    <xacro:if value="${chest_camera}">
+        <link name="openarm_chest_camera_mount"/>
+        <joint name="openarm_chest_camera_mount_joint" type="fixed">
+          <parent link="${chest_camera_parent}"/>
+          <child link="openarm_chest_camera_mount"/>
+          <origin xyz="0 0 0" rpy="0 0 0"/>
+        </joint>
+        <xacro:sensor_d435 parent="openarm_chest_camera_mount" name="chest_camera" use_nominal_extrinsics="true">
+          <origin xyz="${chest_cam_xyz}" rpy="${chest_cam_rpy}"/>
+        </xacro:sensor_d435>
+    </xacro:if>
   </xacro:macro>
 </robot>

File: urdf/robot/v10.urdf.xacro (robot description, xacro)
@@ -35,4 +35,8 @@
   <xacro:arg name="body_cam_xyz" default="0.05 0 0.63"/>
   <xacro:arg name="body_cam_rpy" default="0 ${pi / 6.0} 0"/>
+  <xacro:arg name="chest_camera" default="false"/>
+  <xacro:arg name="chest_cam_xyz" default="0.055 0.045 0.68"/>
+  <xacro:arg name="chest_cam_rpy" default="-2.40 0.03 -1.605"/>
+  <xacro:arg name="chest_camera_parent" default="openarm_link0"/>
   <xacro:arg name="can_fd" default="true" />
   <xacro:openarm_robot
@@ -77,4 +81,8 @@
   body_cam_xyz="$(arg body_cam_xyz)"
   body_cam_rpy="$(arg body_cam_rpy)"
+  chest_camera="$(arg chest_camera)"
+  chest_cam_xyz="$(arg chest_cam_xyz)"
+  chest_cam_rpy="$(arg chest_cam_rpy)"
+  chest_camera_parent="$(arg chest_camera_parent)"
   can_fd="$(arg can_fd)"
   />
